Commit message: Fix differential drive physics and add custom gz-transport bridge
- Fix left/right wheel joint axes to both use Z-axis for symmetric diff drive
- Replace STL wheel collisions with centered cylinders to fix off-center rotation
- Clean left wheel inertia to diagonal (remove SolidWorks off-diagonal terms)
- Add Upper_Swivel damping/friction to prevent continuous free rotation
- Add wheel friction (mu=1.0) via gazebo tags
- Embed robot model in world SDF for persistence across simulation resets
- Add custom cmd_vel_bridge node (gz.transport13) to bypass ros_gz_bridge
  Twist message incompatibility (ignition.msgs vs gz.msgs)
- Set GZ_IP=127.0.0.1 and GZ_SIM_RESOURCE_PATH in launch file

Co-Authored-By: Claude Sonnet 4.6 <noreply@anthropic.com>

File: ros2_ws/src/ass_robot_description/urdf/ASS_Robot.urdf (robot description, URDF)
Before this commit: robot ASS_Robot, 6 links, 5 joints
Links:
- link Castor: geometry collision mesh filename=package://ass_robot_description/meshes/Castor.STL; visual mesh filename=package://ass_robot_description/meshes/Castor.STL
- link Castor_Wheel: geometry collision mesh filename=package://ass_robot_description/meshes/Castor_Wheel.STL; visual mesh filename=package://ass_robot_description/meshes/Castor_Wheel.STL
- link Left_wheel: geometry collision cylinder length=0.05 radius=0.0695; visual mesh filename=package://ass_robot_description/meshes/Left_wheel.STL
- link Right_wheel: geometry collision cylinder length=0.05 radius=0.0695; visual mesh filename=package://ass_robot_description/meshes/Right_wheel.STL
- link Upper_Swivel: geometry collision mesh filename=package://ass_robot_description/meshes/Upper_Swivel.STL; visual mesh filename=package://ass_robot_description/meshes/Upper_Swivel.STL
- link base_link: geometry collision mesh filename=package://ass_robot_description/meshes/base_link.STL; visual mesh filename=package://ass_robot_description/meshes/base_link.STL
Joints:
- removed joint Left_wheel
- removed joint Right_wheel
- added joint left_wheel_joint: type continuous, parent base_link, child Left_wheel, origin xyz=-0.073544 0.24905 -0.1 rpy=-1.5708 0 0, axis 0 0 1
- added joint right_wheel_joint: type continuous, parent base_link, child Right_wheel, origin xyz=-0.073544 -0.24905 -0.1 rpy=-1.5708 0 0, axis 0 0 1

Commit message: Add LiDAR sensor, path follower, and update CLAUDE.md
- Add lidar_link fixed to Upper_Swivel (z+0.3m), 360° CPU lidar sensor
- Add gz-sim-sensors-system plugin to world SDF and regen_world.py template
- Bridge /scan via ros_gz_bridge (LaserScan)
- Add path_follower node: open-loop timed cmd_vel sequence
- Update CLAUDE.md to reflect actual environment (ROS2 Humble, not Jazzy)
  and document all key implementation details

Co-Authored-By: Claude Sonnet 4.6 <noreply@anthropic.com>

File: ros2_ws/src/ass_robot_description/urdf/ASS_Robot.urdf (robot description, URDF)
Before this commit: robot ASS_Robot, 6 links, 5 joints
Links:
- added link lidar_link, mass 0.1; collision cylinder length=0.04 radius=0.05; visual cylinder length=0.04 radius=0.05
Joints:
- added joint lidar_joint: type fixed, parent Upper_Swivel, child lidar_link, origin xyz=0 0 0.3 rpy=0 0 0
